File: Hardware/S2C_motorBoard/Motor.kicad_sch (KiCad schematic)
At the start: 5 parts, among them J301 Moteur, U301 MIC4606, U302 FDMQ86530L

Commit message: PCB update
Parts:
- removed J301: Moteur, Connector_Molex:Molex_CLIK-Mate_502382-0270_1x02-1MP_P1.25mm_Vertical, symbol Connector:Conn_01x02_Pin
- added C201: 2u2, Capacitor_SMD:C_0603_1608Metric, symbol Device:C_Small
- added C204, C205: 10u, Capacitor_SMD:C_0603_1608Metric, symbol Device:C_Small
- added R201, R302: 0R3, Resistor_SMD:R_1210_3225Metric, symbol Device:R_Small
- renumbered C301 to C202, C302 to C203, U302 to U202
Connections:
- net +7.5V: now also C201.1, C204.1, C205.1
- net ARM_A_mes: now also R302.1; no longer U301.10 (AHS)
- net ARM_B_mes: now also R201.1; no longer U301.15 (BHS)
- net GND: now also C201.2, C204.2, C205.2
- net In_A_H renamed In_A
- net In_A_L: no longer names the net of U301.5 (ALI)
- net In_B_H renamed In_B
- net In_B_L: no longer names the net of U301.4 (BLI)
- new net: R302.2, U301.10 (AHS)
- new net: R201.2, U301.15 (BHS)
- no-connect marks 0 -> 2
Other:
- note removed: "Connector"
- moved on the sheet: C202, C203, U301

Commit message: PCB edits
Parts:
- renumbered C201 to C301, C202 to C302, C203 to C303, C204 to C304, C205 to C305, R201 to R301, U202 to U302
Changed lines of the file:
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@@
 		(dnp no)
 		(fields_autoplaced yes)
-		(property "Reference" "#PWR0207"
+		(property "Reference" "#PWR0307"
 			(at 209.55 132.08 0)
 			(effects
@@
 		(on_board yes)
 		(dnp no)
-		(property "Reference" "C204"
+		(property "Reference" "C304"
 			(at 172.72 99.0662 0)
 			(effects
@@
 		(dnp no)
 		(fields_autoplaced yes)
-		(property "Reference" "#PWR0205"
+		(property "Reference" "#PWR0305"
 			(at 179.07 111.76 0)
 			(effects
@@
 		(dnp no)
 		(fields_autoplaced yes)
-		(property "Reference" "#PWR0202"
+		(property "Reference" "#PWR0302"
 			(at 74.93 118.11 0)
 			(effects
@@
 		(dnp no)
 		(fields_autoplaced yes)
-		(property "Reference" "U202"
+		(property "Reference" "U302"
 			(at 211.7441 97.79 0)
 			(effects
@@
 		(on_board yes)
 		(dnp no)
-		(property "Reference" "C201"
+		(property "Reference" "C301"
 			(at 68.58 104.14 0)
 			(effects
@@
 		(dnp no)
 		(fields_autoplaced yes)
-		(property "Reference" "#PWR0203"
+		(property "Reference" "#PWR0303"
 			(at 128.27 116.84 0)
 			(effects
@@
 		(dnp no)
 		(fields_autoplaced yes)
-		(property "Reference" "C203"
+		(property "Reference" "C303"
 			(at 124.4536 93.98 90)
 			(effects
@@
 		(on_board yes)
 		(dnp no)
-		(property "Reference" "#PWR0201"
+		(property "Reference" "#PWR0301"
 			(at 74.93 104.14 0)
 			(effects
@@
 		(dnp no)
 		(fields_autoplaced yes)
-		(property "Reference" "#PWR0204"
+		(property "Reference" "#PWR0304"
 			(at 177.8 99.06 0)
 			(effects
@@
 		(dnp no)
 		(fields_autoplaced yes)
-		(property "Reference" "R201"
+		(property "Reference" "R301"
 			(at 106.68 116.84 90)
 			(effects
@@
 		(dnp no)
 		(fields_autoplaced yes)
-		(property "Reference" "#PWR0206"
+		(property "Reference" "#PWR0306"
 			(at 209.55 99.06 0)
 			(effects
@@
 		(dnp no)
 		(fields_autoplaced yes)
-		(property "Reference" "C205"
+		(property "Reference" "C305"
 			(at 184.15 99.0662 0)
 			(effects
@@
 		(on_board yes)
 		(dnp no)
-		(property "Reference" "C202"
+		(property "Reference" "C302"
 			(at 90.424 120.904 0)
 			(effects

Commit message: last pcb edits
Parts:
- renumbered C301 to C201, C302 to C202, C303 to C203, C304 to C204, C305 to C205, R301 to R201, R302 to R202, U301 to U201, U302 to U202
Changed lines of the file:
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@@
 (kicad_sch
-	(version 20231120)
+	(version 20250114)
 	(generator "eeschema")
-	(generator_version "8.0")
+	(generator_version "9.0")
 	(paper "A4")
+	(rectangle
+		(start 162.56 88.9)
+		(end 241.3 132.08)
+		(stroke
+			(width 0)
+			(type default)
+		)
+		(fill
+			(type none)
+		)
+	)
+	(rectangle
+		(start 66.04 88.9)
+		(end 146.05 132.08)
+		(stroke
+			(width 0)
+			(type default)
+		)
+		(fill
+			(type none)
+		)
+	)
+	(text "Full Bridge\n"
+		(exclude_from_sim no)
+		(at 168.656 90.678 0)
+		(effects
+			(font
+				(size 1.27 1.27)
+			)
+		)
+	)
+	(text "\n"
+		(exclude_from_sim no)
+		(at 95.25 128.27 0)
+		(effects
+			(font
+				(size 1.27 1.27)
+			)
+		)
+	)
+	(text "MOSFET Driver"
+		(exclude_from_sim no)
+		(at 74.168 91.694 0)
+		(effects
+			(font
+				(size 1.27 1.27)
+			)
+		)
+	)
 	(junction
 		(at 177.8 95.25)
@@
 		)
 	)
-	(rectangle
-		(start 162.56 88.9)
-		(end 241.3 132.08)
-		(stroke
-			(width 0)
-			(type default)
-		)
-		(fill
-			(type none)
-		)
-	)
-	(rectangle
-		(start 66.04 88.9)
-		(end 146.05 132.08)
-		(stroke
-			(width 0)
-			(type default)
-		)
-		(fill
-			(type none)
-		)
-	)
-	(text "Full Bridge\n"
-		(exclude_from_sim no)
-		(at 168.656 90.678 0)
-		(effects
-			(font
-				(size 1.27 1.27)
-			)
-		)
-	)
-	(text "\n"
-		(exclude_from_sim no)
-		(at 95.25 128.27 0)
-		(effects
-			(font
-				(size 1.27 1.27)
-			)
-		)
-	)
-	(text "MOSFET Driver"
-		(exclude_from_sim no)
-		(at 74.168 91.694 0)
-		(effects
-			(font
-				(size 1.27 1.27)
-			)
-		)
-	)
 	(label "Cmd_L_B"
 		(at 236.22 116.84 180)
-		(fields_autoplaced yes)
 		(effects
 			(font
@@
 	(label "Cmd_H_B"
 		(at 236.22 106.68 180)
-		(fields_autoplaced yes)
 		(effects
 			(font
@@
 	(label "Cmd_L_A"
 		(at 121.92 107.95 180)
-		(fields_autoplaced yes)
 		(effects
 			(font
@@
 	(label "Cmd_L_A"
 		(at 182.88 116.84 0)
-		(fields_autoplaced yes)
 		(effects
 			(font
@@
 	(label "ARM_B_mes"
 		(at 123.19 121.92 180)
-		(fields_autoplaced yes)
 		(effects
 			(font
@@
 	(label "ARM_A_mes"
 		(at 182.88 111.76 0)
-		(fields_autoplaced yes)
 		(effects
 			(font
@@
 	(label "ARM_A_mes"
 		(at 140.97 105.41 180)
-		(fields_autoplaced yes)
 		(effects
 			(font
@@
 	(label "Cmd_H_A"
 		(at 182.88 106.68 0)
-		(fields_autoplaced yes)
 		(effects
 			(font
@@
 	(label "ARM_A_mes"
 		(at 138.43 100.33 180)
-		(fields_autoplaced yes)
 		(effects
 			(font
@@
 	(label "Cmd_H_A"
 		(at 121.92 102.87 180)
-		(fields_autoplaced yes)
 		(effects
 			(font
@@
 	(label "Cmd_H_B"
 		(at 107.95 128.27 180)
-		(fields_autoplaced yes)
 		(effects
 			(font
@@
 	(label "ARM_B_mes"
 		(at 83.82 128.27 0)
-		(fields_autoplaced yes)
 		(effects
 			(font
@@
 	(label "Cmd_L_B"
 		(at 124.46 113.03 180)
-		(fields_autoplaced yes)
 		(effects
 			(font
@@
 	(label "ARM_B_mes"
 		(at 236.22 111.76 180)
-		(fields_autoplaced yes)
 		(effects
 			(font
@@
 		(shape input)
 		(at 85.09 110.49 180)
-		(fields_autoplaced yes)
 		(effects
 			(font
@@
 		(shape input)
 		(at 228.6 114.3 0)
-		(fields_autoplaced yes)
 		(effects
 			(font
@@
 		(shape input)
 		(at 190.5 114.3 180)
-		(fields_autoplaced yes)
 		(effects
 			(font
@@
 		(shape input)
 		(at 85.09 105.41 180)
-		(fields_autoplaced yes)
 		(effects
 			(font
@@
 		(dnp no)
 		(fields_autoplaced yes)
-		(property "Reference" "#PWR0307"
+		(property "Reference" "#PWR0207"
 			(at 209.55 132.08 0)
 			(effects
@@
 		(on_board yes)
 		(dnp no)
-		(property "Reference" "C304"
+		(property "Reference" "C204"
 			(at 172.72 99.0662 0)
 			(effects
@@
 		(dnp no)
 		(fields_autoplaced yes)
-		(property "Reference" "#PWR0305"
+		(property "Reference" "#PWR0205"
 			(at 179.07 111.76 0)
 			(effects
@@
 		(dnp no)
 		(fields_autoplaced yes)
-		(property "Reference" "#PWR0302"
+		(property "Reference" "#PWR0202"
 			(at 74.93 118.11 0)
 			(effects
@@
 		(dnp no)
 		(fields_autoplaced yes)
-		(property "Reference" "U302"
+		(property "Reference" "U202"
 			(at 211.7441 97.79 0)
 			(effects
@@
 		(on_board yes)
 		(dnp no)
-		(property "Reference" "C301"
+		(property "Reference" "C201"
 			(at 68.58 104.14 0)
 			(effects
@@
 		(dnp no)
 		(fields_autoplaced yes)
-		(property "Reference" "#PWR0303"
+		(property "Reference" "#PWR0203"
 			(at 128.27 116.84 0)
 			(effects
@@
 		(dnp no)
 		(fields_autoplaced yes)
-		(property "Reference" "C303"
+		(property "Reference" "C203"
 			(at 124.4536 93.98 90)
 			(effects
@@
 		(on_board yes)
 		(dnp no)
-		(property "Reference" "#PWR0301"
+		(property "Reference" "#PWR0201"
 			(at 74.93 104.14 0)
 			(effects
@@
 		(dnp no)
 		(fields_autoplaced yes)
-		(property "Reference" "#PWR0304"
+		(property "Reference" "#PWR0204"
 			(at 177.8 99.06 0)
 			(effects
@@
 		(on_board yes)
 		(dnp no)
-		(property "Reference" "R302"
+		(property "Reference" "R202"
 			(at 131.318 106.934 90)
 			(effects
@@
 		(dnp no)
 		(fields_autoplaced yes)
-		(property "Reference" "R301"
+		(property "Reference" "R201"
 			(at 106.68 116.84 90)
 			(effects
@@
 		(dnp no)
 		(fields_autoplaced yes)
-		(property "Reference" "#PWR0306"
+		(property "Reference" "#PWR0206"
 			(at 209.55 99.06 0)
 			(effects
@@
 		(dnp no)
 		(fields_autoplaced yes)
-		(property "Reference" "C305"
+		(property "Reference" "C205"
 			(at 184.15 99.0662 0)
 			(effects
@@
 		(on_board yes)
 		(dnp no)
-		(property "Reference" "C302"
+		(property "Reference" "C202"
 			(at 90.424 120.904 0)
 			(effects
@@
 		(dnp no)
 		(fields_autoplaced yes)
-		(property "Reference" "U301"
+		(property "Reference" "U201"
 			(at 99.06 93.98 0)
 			(effects
