File: Hardware/S2C_motorBoard/S2C_motorBoard.kicad_sch (KiCad schematic)
At the start: 30 parts, among them J101 UART, J102 Conn_ST_STDC14, J103 USB_C_Receptacle_USB2.0_16P, U101 WPME-VDLM, U102 STM32G431CBUx, U103 USBLC6-2SC6

Commit message: PCB update
Parts:
- removed L101: 39n, Inductor_SMD:L_0603_1608Metric, symbol Device:L_Small
- added J101: Conn_02x04_Odd_Even, Connector_Molex:Molex_Mini-Fit_Jr_5566-08A_2x04_P4.20mm_Vertical, symbol Connector_Generic:Conn_02x04_Top_Bottom
- C110: renamed from C106; footprint Capacitor_SMD:C_0603_1608Metric_Pad1.08x0.95mm_HandSolder -> Capacitor_SMD:C_0603_1608Metric
- TP101: footprint TestPoint:TestPoint_Pad_2.0x2.0mm -> TestPoint:TestPoint_Pad_D2.0mm
- renumbered C105 to C104, C104 to C105, C107 to C106, C109 to C107, C111 to C108, C112 to C109, C108 to C111, C110 to C112, H104 to H101, H103 to H102, H102 to H103, H101 to H104, J101 to J102, J102 to J103, J103 to J104
Connections:
- net +3.3VA is gone; now on net +3.3V: C110.1, C111.1, C112.1, U102.20 (VREF+), U102.21 (VDDA)
- net +7.5V: now also BT101.2 (+); no longer BT101.1 (+)
- net D+: now also U103.6 (I/O1); no longer U103.1 (I/O1)
- net D-: now also U103.4 (I/O2); no longer U103.6 (I/O1)
- net GND: now also BT101.1 (-); no longer BT101.2 (-)
- net USB_DN: now also U103.3 (I/O2); no longer U103.4 (I/O2)
- net USB_DP: now also U103.1 (I/O1); no longer U103.3 (I/O2)
- net M3_In_A: now reaches U102.10 (PA2)
- net M3_In_B: now reaches U102.11 (PA3)
- net M1_In_B: now reaches U102.46 (PB8)
- net M1_In_A: now reaches U102.47 (PB9)
- net M2_In_A: now reaches U102.8 (PA0)
- net M2_In_B: now reaches U102.9 (PA1)
- net M1_In_A_H: no longer names the net of U102.16 (PC4)
- net M1_In_A_L renamed M4_In_B
- net M1_In_B_H: no longer names the net of U102.13 (PA5)
- net M1_In_B_L renamed M4_In_A
- net M2_In_A_H: no longer names the net of U102.42 (PB4)
- net M2_In_A_L: no longer names the net of U102.43 (PB5)
- net M2_In_B_H: no longer names the net of U102.45 (PB7)
- net M2_In_B_L: no longer names the net of U102.44 (PB6)
- new net M1_ARM_A: J101.8 (Pin_8)
- new net M1_ARM_B: J101.4 (Pin_4)
- new net M2_ARM_A: J101.7 (Pin_7)
- new net M2_ARM_B: J101.3 (Pin_3)
- new net M3_ARM_A: J101.6 (Pin_6)
- new net M3_ARM_B: J101.2 (Pin_2)
- new net M4_ARM_A: J101.5 (Pin_5)
- new net M4_ARM_B: J101.1 (Pin_1)
Other:
- added sheet Motor3 (Motor.kicad_sch)
- added sheet Motor4 (Motor.kicad_sch)
- sheet Motor1 ports: added ARM_A, ARM_B, In_A, In_B; removed In_A_H, In_A_L, In_B_H, In_B_L
- sheet Motor2 ports: added ARM_A, ARM_B, In_A, In_B; removed In_A_H, In_A_L, In_B_H, In_B_L
- note added: "Connector"
- moved on the sheet: BT101, C101, C102, C103, C104, C106, C107, C108, C109, C110, C111, C112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

Commit message: PCB edits
Parts:
- added R1: 10k, Resistor_SMD:R_0402_1005Metric, symbol Device:R_Small
Connections:
- net GND: now also R1.2
- net M1_In_A: now also U102.45 (PB7); no longer U102.47 (PB9)
- net M1_In_B: now also U102.44 (PB6); no longer U102.46 (PB8)
- new net: R1.1, U102.46 (PB8)
- no-connect marks 33 -> 32
